Commit message: customize lidar

File: velodyne_description/urdf/example.urdf.xacro (robot description, xacro)
@@ -32,11 +32,7 @@
     </inertial>
   </link>
-  <xacro:include filename="$(find velodyne_description)/urdf/VLP-16.urdf.xacro"/>
-  <xacro:VLP-16 parent="base_link" name="velodyne" topic="/velodyne_points" organize_cloud="${organize_cloud}" hz="10" samples="440" gpu="${gpu}">
+  <xacro:include filename="$(find velodyne_description)/urdf/RS-Helios-5515.urdf.xacro"/>
+  <xacro:RS-Helios-5515 parent="base_link" name="rs_helios" topic="/rslidar_points" organize_cloud="${organize_cloud}" hz="10" samples="220" gpu="${gpu}">
     <origin xyz="0 0 0.4" rpy="0 0 0" />
-  </xacro:VLP-16>
-  <xacro:include filename="$(find velodyne_description)/urdf/HDL-32E.urdf.xacro"/>
-  <xacro:HDL-32E parent="base_link" name="velodyne2" topic="/velodyne_points2" organize_cloud="${organize_cloud}" hz="10" samples="220" gpu="${gpu}">
-    <origin xyz="0 0 0.6" rpy="0 0 0" />
-  </xacro:HDL-32E>
+  </xacro:RS-Helios-5515>
 </robot>

Commit message: add imu and some boxes for simulation

File: velodyne_description/urdf/example.urdf.xacro (robot description, xacro)
@@ -32,4 +32,8 @@
     </inertial>
   </link>
+  <xacro:include filename="$(find velodyne_description)/urdf/imu.urdf.xacro"/>
+  <xacro:imu parent="base_link" name="imu_link" topic="/imu">
+    <origin xyz="0 0 0" rpy="0 0 0" />
+  </xacro:imu>
   <xacro:include filename="$(find velodyne_description)/urdf/RS-Helios-5515.urdf.xacro"/>
   <xacro:RS-Helios-5515 parent="base_link" name="rslidar" topic="/rslidar_points" organize_cloud="${organize_cloud}" hz="10" samples="1800" gpu="${gpu}">
