Commit message: make same topic hear like unitree lidar

File: velodyne_description/urdf/RS-Helios-5515.urdf.xacro (robot description, xacro)
@@ -3,5 +3,5 @@
   <xacro:property name="M_PI" value="3.1415926535897931" />
   <!-- RoboSense RS-Helios 5515: 32-channel, 360° horizontal, -55° to +15° vertical FOV -->
-  <xacro:macro name="RS-Helios-5515" params="*origin parent:=base_link name:=rs_helios tf_prefix:='' topic:=/rslidar_points organize_cloud:=false hz:=10 lasers:=32 samples:=1800 collision_range:=0.2 min_range:=0.2 max_range:=150.0 noise:=0.008 min_angle:=-${M_PI} max_angle:=${M_PI} gpu:=false">
+  <xacro:macro name="RS-Helios-5515" params="*origin parent:=base_link name:=rslidar tf_prefix:='' topic:=/rslidar_points organize_cloud:=true hz:=10 lasers:=32 samples:=1800 collision_range:=0.2 min_range:=0.2 max_range:=150.0 noise:=0.008 min_angle:=-${M_PI} max_angle:=${M_PI} gpu:=false">
     <joint name="${name}_base_mount_joint" type="fixed">
       <xacro:insert_block name="origin" />

File: velodyne_description/urdf/example.urdf.xacro (robot description, xacro)
@@ -3,5 +3,5 @@
   <xacro:arg name="gpu" default="false"/>
   <xacro:property name="gpu" value="$(arg gpu)" />
-  <xacro:arg name="organize_cloud" default="false"/>
+  <xacro:arg name="organize_cloud" default="true"/>
   <xacro:property name="organize_cloud" value="$(arg organize_cloud)" />
   <!-- Base Footprint -->
@@ -33,5 +33,5 @@
   </link>
   <xacro:include filename="$(find velodyne_description)/urdf/RS-Helios-5515.urdf.xacro"/>
-  <xacro:RS-Helios-5515 parent="base_link" name="rs_helios" topic="/rslidar_points" organize_cloud="${organize_cloud}" hz="10" samples="220" gpu="${gpu}">
+  <xacro:RS-Helios-5515 parent="base_link" name="rslidar" topic="/rslidar_points" organize_cloud="${organize_cloud}" hz="10" samples="1800" gpu="${gpu}">
     <origin xyz="0 0 0.4" rpy="0 0 0" />
   </xacro:RS-Helios-5515>

Commit message: update cpu ray sensor speed and intensity logic

File: velodyne_description/urdf/RS-Helios-5515.urdf.xacro (robot description, xacro)
@@ -3,5 +3,5 @@
   <xacro:property name="M_PI" value="3.1415926535897931" />
   <!-- RoboSense RS-Helios 5515: 32-channel, 360° horizontal, -55° to +15° vertical FOV -->
-  <xacro:macro name="RS-Helios-5515" params="*origin parent:=base_link name:=rslidar tf_prefix:='' topic:=/rslidar_points organize_cloud:=true hz:=10 lasers:=32 samples:=1800 collision_range:=0.2 min_range:=0.2 max_range:=150.0 noise:=0.008 min_angle:=-${M_PI} max_angle:=${M_PI} gpu:=false">
+  <xacro:macro name="RS-Helios-5515" params="*origin parent:=base_link name:=rslidar tf_prefix:='' topic:=/rslidar_points organize_cloud:=true hz:=10 lasers:=32 samples:=1800 collision_range:=0.2 min_range:=0.2 max_range:=150.0 noise:=0.008 min_angle:=-${M_PI} max_angle:=${M_PI} gpu:=false threads:=0">
     <joint name="${name}_base_mount_joint" type="fixed">
       <xacro:insert_block name="origin" />
@@ -94,4 +94,5 @@
             <max_range>${max_range}</max_range>
             <gaussian_noise>${noise}</gaussian_noise>
+            <threads>${threads}</threads>
           </plugin>
         </sensor>
@@ -139,4 +140,5 @@
             <max_range>${max_range}</max_range>
             <gaussian_noise>${noise}</gaussian_noise>
+            <threads>${threads}</threads>
           </plugin>
         </sensor>
